File: hardware/racer/racer.kicad_sch (KiCad schematic)
At the start: 79 parts, among them J1 motor0, J11 UART, J12 JST 2.0 BATT, J2 motor1, J3 motor0, J4 motor1, J5 motor0, J6 motor1, J7 motor0, J8 motor1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

Commit message: fix(lcsc): Starting to add LCSC part numbers
Parts:
- C1, C15, C16, C2, C5, C6: LCSC (none) -> C19702
- C10: LCSC (none) -> C15849
- C12, C13, C3, C4, C7, C8: LCSC (none) -> C14663
- C9: LCSC (none) -> C178330
- R1, R10, R11, R3, R30, R5, R7, R9: LCSC (none) -> C25804
- R12, R13, R14, R15, R20, R21, R25: LCSC (none) -> C8218
- R16: LCSC (none) -> C22935
- R17, R18: LCSC (none) -> C23186
- R2, R4, R6, R8: LCSC (none) -> C22984
- R24: LCSC (none) -> C23242
- R26, R27, R28, R29: LCSC (none) -> C25803
- U5: LCSC (none) -> C18202993
- U6: LCSC (none) -> C20627184

Commit message: fix(changes): More LCSC numbers added
Parts:
- C11: LCSC (none) -> C14663
- C14: LCSC (none) -> C23630
- C17: LCSC (none) -> C59461
- D1, D2, D6, D8, D9: LCSC (none) -> C2286
- D3, D4: LCSC (none) -> C2290
- D5: LCSC (none) -> C314264
- J11: LCSC (none) -> C7430360
- J12: LCSC (none) -> C594142
- S2, S3: LCSC (none) -> C455282
- TH1: LCSC (none) -> C13564
- U7: LCSC (none) -> C627668
Changed lines of the file:
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@@
 			)
 		)
+		(property "LCSC" "C455282"
+			(at 140.335 340.995 90)
+			(effects
+				(font
+					(size 1.27 1.27)
+				)
+				(hide yes)
+			)
+		)
 		(pin "1"
 		)
@@
 			)
 		)
+		(property "LCSC" "C314264"
+			(at 178.435 114.935 0)
+			(effects
+				(font
+					(size 1.27 1.27)
+				)
+				(hide yes)
+			)
+		)
 		(pin "1"
 		)
@@
 			)
 		)
+		(property "LCSC" "C2286"
+			(at 241.3 170.18 0)
+			(effects
+				(font
+					(size 1.27 1.27)
+				)
+				(hide yes)
+			)
+		)
 		(pin "1"
 		)
@@
 			)
 		)
+		(property "LCSC" "C455282"
+			(at 200.025 325.12 90)
+			(effects
+				(font
+					(size 1.27 1.27)
+				)
+				(hide yes)
+			)
+		)
 		(pin "1"
 		)
@@
 			)
 		)
+		(property "LCSC" "C14663"
+			(at 118.745 257.175 0)
+			(effects
+				(font
+					(size 1.27 1.27)
+				)
+				(hide yes)
+			)
+		)
 		(pin "1"
 		)
@@
 			)
 		)
+		(property "LCSC" "C13564"
+			(at 266.7 129.54 0)
+			(effects
+				(font
+					(size 1.27 1.27)
+				)
+				(hide yes)
+			)
+		)
 		(pin "1"
 		)
@@
 			)
 		)
+		(property "LCSC" "C2286"
+			(at 311.785 86.995 0)
+			(effects
+				(font
+					(size 1.27 1.27)
+				)
+				(hide yes)
+			)
+		)
 		(pin "2"
 		)
@@
 			)
 		)
+		(property "LCSC" "C23630"
+			(at 340.995 89.535 0)
+			(effects
+				(font
+					(size 1.27 1.27)
+				)
+				(hide yes)
+			)
+		)
 		(pin "1"
 		)
@@
 			)
 		)
+		(property "LCSC" "C2290"
+			(at 280.035 282.575 0)
+			(effects
+				(font
+					(size 1.27 1.27)
+				)
+				(hide yes)
+			)
+		)
 		(pin "1"
 		)
@@
 			)
 		)
+		(property "LCSC" "C2286"
+			(at 280.035 264.795 0)
+			(effects
+				(font
+					(size 1.27 1.27)
+				)
+				(hide yes)
+			)
+		)
 		(pin "1"
 		)
@@
 			)
 		)
+		(property "LCSC" "C59461"
+			(at 275.59 115.57 0)
+			(effects
+				(font
+					(size 1.27 1.27)
+				)
+				(hide yes)
+			)
+		)
 		(pin "1"
 		)
@@
 			)
 		)
+		(property "LCSC" "C2286"
+			(at 248.92 170.18 0)
+			(effects
+				(font
+					(size 1.27 1.27)
+				)
+				(hide yes)
+			)
+		)
 		(pin "1"
 		)
@@
 			)
 		)
+		(property "LCSC" "C2286"
+			(at 280.035 273.685 0)
+			(effects
+				(font
+					(size 1.27 1.27)
+				)
+				(hide yes)
+			)
+		)
 		(pin "1"
 		)
@@
 			)
 		)
+		(property "LCSC" "C7430360"
+			(at 239.395 219.075 90)
+			(effects
+				(font
+					(size 1.27 1.27)
+				)
+				(hide yes)
+			)
+		)
 		(pin "1"
 		)
@@
 			)
 		)
+		(property "LCSC" "C594142"
+			(at 263.525 56.515 90)
+			(effects
+				(font
+					(size 1.27 1.27)
+				)
+				(hide yes)
+			)
+		)
 		(pin "1"
 		)
@@
 			)
 		)
+		(property "LCSC" "C2290"
+			(at 280.035 291.465 0)
+			(effects
+				(font
+					(size 1.27 1.27)
+				)
+				(hide yes)
+			)
+		)
 		(pin "1"
 		)
@@
 			(at 242.57 114.3 0)
 			(effects
+				(font
+					(size 1.27 1.27)
+				)
+				(hide yes)
+			)
+		)
+		(property "LCSC" "C627668"
+			(at 242.57 114.3 0)
+			(effects
